Commit message: fix: PCA9685 clock correction and controller startup issues
- Add configurable clock_correction parameter for PCA9685 oscillator drift
  (xacro param, no rebuild needed when changing boards)
- Fix controller namespace matching with /**/ prefix in YAML
- Remove empty joint_state_broadcaster config causing crash
- Add minimal URDF links/joints for robot_state_publisher

File: config/minicar_ackermann_real.xacro (robot description, xacro)
@@ -1,6 +1,30 @@
 <?xml version="1.0"?>
 <robot xmlns:xacro="http://www.ros.org/wiki/xacro" name="minicar_ackermann_real">
-  <!-- Include base URDF from simulation package -->
-  <!-- Note: You may need to create a separate hardware-specific URDF or reuse simulation URDF -->
+  <!-- Launch arguments -->
+  <xacro:arg name="robot_ns" default="real_robot"/>
+  <!-- Minimal robot structure for hardware interface -->
+  <link name="base_link"/>
+  <link name="rear_left_wheel"/>
+  <link name="rear_right_wheel"/>
+  <link name="front_left_steering"/>
+  <link name="front_right_steering"/>
+  <joint name="rear_left_wheel_joint" type="continuous">
+    <parent link="base_link"/>
+    <child link="rear_left_wheel"/>
+  </joint>
+  <joint name="rear_right_wheel_joint" type="continuous">
+    <parent link="base_link"/>
+    <child link="rear_right_wheel"/>
+  </joint>
+  <joint name="front_left_steering_joint" type="revolute">
+    <parent link="base_link"/>
+    <child link="front_left_steering"/>
+    <limit lower="-0.5236" upper="0.5236" effort="10" velocity="1.0"/>
+  </joint>
+  <joint name="front_right_steering_joint" type="revolute">
+    <parent link="base_link"/>
+    <child link="front_right_steering"/>
+    <limit lower="-0.5236" upper="0.5236" effort="10" velocity="1.0"/>
+  </joint>
   <!-- ros2_control hardware interface definition -->
   <ros2_control name="AckermannRealSystem" type="system">
@@ -19,4 +43,6 @@
       <param name="servo_center_pulse_ms">1.5</param>
       <param name="servo_max_pulse_ms">2.0</param>
+      <!-- PCA9685 Clock Correction (per-board oscillator drift) -->
+      <param name="clock_correction">1.1</param>
       <!-- ESC Calibration (adjust based on actual ESC) -->
       <param name="esc_min_pulse_ms">1.0</param>
